File: kicad/Row_A.sch (KiCad schematic (older format))
At the start: 68 parts, among them U1 APA102, U10 APA102, U11 APA102, U12 APA102, U13 APA102, U14 APA102, U15 APA102, U16 APA102, U17 APA102, U18 APA102, U19 APA102, U2 APA102, U20 APA102, U21 APA102, U22 APA102, U23 APA102, U24 APA102, U25 APA102, U26 APA102, U27 APA102, U28 APA102, U29 APA102, U3 APA102, U30 APA102, U31 APA102, U32 APA102, U33 APA102, U34 APA102, U35 APA102, U36 APA102, U37 APA102, U38 APA102, U39 APA102, U4 APA102, U40 APA102, U41 APA102, U42 APA102, U43 APA102, U44 APA102, U45 APA102, U46 APA102, U47 APA102, U48 APA102, U49 APA102, U5 APA102, U50 APA102, U51 APA102, U52 APA102, U53 APA102, U54 APA102, U55 APA102, U56 APA102, U57 APA102, U58 APA102, U59 APA102, U6 APA102, U60 APA102, U61 APA102, U62 APA102, U63 APA102, U64 APA102, U7 APA102, U8 APA102, U9 APA102

Commit message: WIP
Parts:
- added P5: GND, ultim8x64_libs:PowerIn_stud, symbol CONN_1
- added P6: 5V, ultim8x64_libs:PowerIn_stud, symbol CONN_1
- C1, C2: footprint ultim8x8_libs:c_2917 -> ultim8x64_libs:c_2917
- C3, C4: footprint ultim8x8_libs:c_0805 -> ultim8x64_libs:c_0805
- U1, U10, U15, U16, U17, U18, U2, U20, U23, U24, U25, U26, U27, U28, U3, U31, U32, U33, U34, U35, U36, U39, U4, U40, U41, U42, U44, U47, U48, U49, U50, U51, U52, U55, U56, U57, U58, U63, U64, U7, U8, U9: footprint ultim8x8_libs:APA102 -> ultim8x64_libs:APA102
- U11: footprint ultim8x8_libs:APA102 -> ultim8x64_libs:APA102_U11
- U12: footprint ultim8x8_libs:APA102 -> ultim8x64_libs:APA102_U12
- U13, U21, U29, U37, U45, U61: footprint ultim8x8_libs:APA102_U05 -> ultim8x64_libs:APA102
- U14, U22, U30, U46, U62: footprint ultim8x8_libs:APA102_U06 -> ultim8x64_libs:APA102
- U19: footprint ultim8x8_libs:APA102 -> ultim8x64_libs:APA102_U19
- U38: footprint ultim8x8_libs:APA102_U06 -> ultim8x64_libs:APA102_U38
- U43: footprint ultim8x8_libs:APA102 -> ultim8x64_libs:APA102_U43
- U5: footprint ultim8x8_libs:APA102 -> ultim8x64_libs:APA102_U05
- U53: footprint ultim8x8_libs:APA102_U05 -> ultim8x64_libs:APA102_U53
- U54: footprint ultim8x8_libs:APA102_U06 -> ultim8x64_libs:APA102_U54
- U59: footprint ultim8x8_libs:APA102 -> ultim8x64_libs:APA102_U59
- U6: footprint ultim8x8_libs:APA102 -> ultim8x64_libs:APA102_U06
- U60: footprint ultim8x8_libs:APA102 -> ultim8x64_libs:APA102_U60
Connections:
- net 5V: now also C1.1 (+), C2.1 (+), C3.1, C4.1, P5.1
- net GND: now also C1.2 (-), C2.2 (-), C3.2, C4.2, P6.1
Other:
- note added: "POWER INPUT POSTS"
