File: kicad/Row_B.sch (KiCad schematic (older format))
At the start: 68 parts, among them U100 APA102, U101 APA102, U102 APA102, U103 APA102, U104 APA102, U105 APA102, U106 APA102, U107 APA102, U108 APA102, U109 APA102, U110 APA102, U111 APA102, U112 APA102, U113 APA102, U114 APA102, U115 APA102, U116 APA102, U117 APA102, U118 APA102, U119 APA102, U120 APA102, U121 APA102, U122 APA102, U123 APA102, U124 APA102, U125 APA102, U126 APA102, U127 APA102, U128 APA102, U65 APA102, U66 APA102, U67 APA102, U68 APA102, U69 APA102, U70 APA102, U71 APA102, U72 APA102, U73 APA102, U74 APA102, U75 APA102, U76 APA102, U77 APA102, U78 APA102, U79 APA102, U80 APA102, U81 APA102, U82 APA102, U83 APA102, U84 APA102, U85 APA102, U86 APA102, U87 APA102, U88 APA102, U89 APA102, U90 APA102, U91 APA102, U92 APA102, U93 APA102, U94 APA102, U95 APA102, U96 APA102, U97 APA102, U98 APA102, U99 APA102

Commit message: WIP
Parts:
- C5, C6: footprint ultim8x8_libs:c_2917 -> ultim8x64_libs:c_2917
- C7, C8: footprint ultim8x8_libs:c_0805 -> ultim8x64_libs:c_0805
- U100, U103, U104, U105, U106, U107, U108, U111, U112, U113, U114, U115, U116, U119, U120, U121, U122, U123, U124, U127, U128, U65, U66, U67, U68, U69, U70, U71, U72, U73, U74, U75, U76, U79, U80, U81, U82, U83, U84, U87, U88, U89, U90, U91, U92, U95, U96, U97, U98, U99: footprint ultim8x8_libs:APA102 -> ultim8x64_libs:APA102
- U101, U109, U117, U125, U77, U85, U93: footprint ultim8x8_libs:APA102_U05 -> ultim8x64_libs:APA102
- U102, U110, U118, U126, U78, U86, U94: footprint ultim8x8_libs:APA102_U06 -> ultim8x64_libs:APA102
