File: kicad/Row_C.sch (KiCad schematic (older format))
At the start: 68 parts, among them U129 APA102, U130 APA102, U131 APA102, U132 APA102, U133 APA102, U134 APA102, U135 APA102, U136 APA102, U137 APA102, U138 APA102, U139 APA102, U140 APA102, U141 APA102, U142 APA102, U143 APA102, U144 APA102, U145 APA102, U146 APA102, U147 APA102, U148 APA102, U149 APA102, U150 APA102, U151 APA102, U152 APA102, U153 APA102, U154 APA102, U155 APA102, U156 APA102, U157 APA102, U158 APA102, U159 APA102, U160 APA102, U161 APA102, U162 APA102, U163 APA102, U164 APA102, U165 APA102, U166 APA102, U167 APA102, U168 APA102, U169 APA102, U170 APA102, U171 APA102, U172 APA102, U173 APA102, U174 APA102, U175 APA102, U176 APA102, U177 APA102, U178 APA102, U179 APA102, U180 APA102, U181 APA102, U182 APA102, U183 APA102, U184 APA102, U185 APA102, U186 APA102, U187 APA102, U188 APA102, U189 APA102, U190 APA102, U191 APA102, U192 APA102

Commit message: WIP
Parts:
- added P7: GND, ultim8x64_libs:PowerIn_stud, symbol CONN_1
- added P8: 5V, ultim8x64_libs:PowerIn_stud, symbol CONN_1
- C10, C9: footprint ultim8x8_libs:c_2917 -> ultim8x64_libs:c_2917
- C11, C12: footprint ultim8x8_libs:c_0805 -> ultim8x64_libs:c_0805
- U129, U130, U131, U132, U135, U136, U137, U138, U143, U144, U145, U146, U148, U151, U152, U153, U154, U155, U156, U159, U160, U161, U162, U163, U164, U167, U168, U169, U170, U172, U175, U176, U177, U178, U179, U180, U183, U184, U185, U186, U191, U192: footprint ultim8x8_libs:APA102 -> ultim8x64_libs:APA102
- U133: footprint ultim8x8_libs:APA102 -> ultim8x64_libs:APA102_U05
- U134: footprint ultim8x8_libs:APA102 -> ultim8x64_libs:APA102_U06
- U139: footprint ultim8x8_libs:APA102 -> ultim8x64_libs:APA102_U11
- U140: footprint ultim8x8_libs:APA102 -> ultim8x64_libs:APA102_U12
- U141, U149, U157, U165, U173, U189: footprint ultim8x8_libs:APA102_U05 -> ultim8x64_libs:APA102
- U142, U150, U158, U174, U190: footprint ultim8x8_libs:APA102_U06 -> ultim8x64_libs:APA102
- U147: footprint ultim8x8_libs:APA102 -> ultim8x64_libs:APA102_U19
- U166: footprint ultim8x8_libs:APA102_U06 -> ultim8x64_libs:APA102_U38
- U171: footprint ultim8x8_libs:APA102 -> ultim8x64_libs:APA102_U43
- U181: footprint ultim8x8_libs:APA102_U05 -> ultim8x64_libs:APA102_U53
- U182: footprint ultim8x8_libs:APA102_U06 -> ultim8x64_libs:APA102_U54
- U187: footprint ultim8x8_libs:APA102 -> ultim8x64_libs:APA102_U59
- U188: footprint ultim8x8_libs:APA102 -> ultim8x64_libs:APA102_U60
Connections:
- net 5V: now also C10.1 (+), C11.1, C12.1, C9.1 (+), P7.1
- net GND: now also C10.2 (-), C11.2, C12.2, C9.2 (-), P8.1
Other:
- note added: "POWER INPUT POSTS"
