File: kicad/Row_D.sch (KiCad schematic (older format))
At the start: 68 parts, among them U193 APA102, U194 APA102, U195 APA102, U196 APA102, U197 APA102, U198 APA102, U199 APA102, U200 APA102, U201 APA102, U202 APA102, U203 APA102, U204 APA102, U205 APA102, U206 APA102, U207 APA102, U208 APA102, U209 APA102, U210 APA102, U211 APA102, U212 APA102, U213 APA102, U214 APA102, U215 APA102, U216 APA102, U217 APA102, U218 APA102, U219 APA102, U220 APA102, U221 APA102, U222 APA102, U223 APA102, U224 APA102, U225 APA102, U226 APA102, U227 APA102, U228 APA102, U229 APA102, U230 APA102, U231 APA102, U232 APA102, U233 APA102, U234 APA102, U235 APA102, U236 APA102, U237 APA102, U238 APA102, U239 APA102, U240 APA102, U241 APA102, U242 APA102, U243 APA102, U244 APA102, U245 APA102, U246 APA102, U247 APA102, U248 APA102, U249 APA102, U250 APA102, U251 APA102, U252 APA102, U253 APA102, U254 APA102, U255 APA102, U256 APA102

Commit message: WIP
Parts:
- C13, C14: footprint ultim8x8_libs:c_2917 -> ultim8x64_libs:c_2917
- C15, C16: footprint ultim8x8_libs:c_0805 -> ultim8x64_libs:c_0805
- U193, U194, U195, U196, U197, U198, U199, U200, U201, U202, U203, U204, U207, U208, U209, U210, U211, U212, U215, U216, U217, U218, U219, U220, U223, U224, U225, U226, U227, U228, U231, U232, U233, U234, U235, U236, U239, U240, U241, U242, U243, U244, U247, U248, U249, U250, U251, U252, U255, U256: footprint ultim8x8_libs:APA102 -> ultim8x64_libs:APA102
- U205, U213, U221, U229, U237, U245, U253: footprint ultim8x8_libs:APA102_U05 -> ultim8x64_libs:APA102
- U206, U214, U222, U230, U238, U246, U254: footprint ultim8x8_libs:APA102_U06 -> ultim8x64_libs:APA102
