File: kicad/Row_E.sch (KiCad schematic (older format))
At the start: 68 parts, among them U257 APA102, U258 APA102, U259 APA102, U260 APA102, U261 APA102, U262 APA102, U263 APA102, U264 APA102, U265 APA102, U266 APA102, U267 APA102, U268 APA102, U269 APA102, U270 APA102, U271 APA102, U272 APA102, U273 APA102, U274 APA102, U275 APA102, U276 APA102, U277 APA102, U278 APA102, U279 APA102, U280 APA102, U281 APA102, U282 APA102, U283 APA102, U284 APA102, U285 APA102, U286 APA102, U287 APA102, U288 APA102, U289 APA102, U290 APA102, U291 APA102, U292 APA102, U293 APA102, U294 APA102, U295 APA102, U296 APA102, U297 APA102, U298 APA102, U299 APA102, U300 APA102, U301 APA102, U302 APA102, U303 APA102, U304 APA102, U305 APA102, U306 APA102, U307 APA102, U308 APA102, U309 APA102, U310 APA102, U311 APA102, U312 APA102, U313 APA102, U314 APA102, U315 APA102, U316 APA102, U317 APA102, U318 APA102, U319 APA102, U320 APA102

Commit message: WIP
Parts:
- added P10: 5V, ultim8x64_libs:PowerIn_stud, symbol CONN_1
- added P9: GND, ultim8x64_libs:PowerIn_stud, symbol CONN_1
- C17, C18: footprint ultim8x8_libs:c_2917 -> ultim8x64_libs:c_2917
- C19, C20: footprint ultim8x8_libs:c_0805 -> ultim8x64_libs:c_0805
- U257, U258, U259, U260, U263, U264, U265, U266, U271, U272, U273, U274, U276, U279, U280, U281, U282, U283, U284, U287, U288, U289, U290, U291, U292, U295, U296, U297, U298, U300, U303, U304, U305, U306, U307, U308, U311, U312, U313, U314, U319, U320: footprint ultim8x8_libs:APA102 -> ultim8x64_libs:APA102
- U261: footprint ultim8x8_libs:APA102 -> ultim8x64_libs:APA102_U05
- U262: footprint ultim8x8_libs:APA102 -> ultim8x64_libs:APA102_U06
- U267: footprint ultim8x8_libs:APA102 -> ultim8x64_libs:APA102_U11
- U268: footprint ultim8x8_libs:APA102 -> ultim8x64_libs:APA102_U12
- U269, U277, U285, U293, U301, U317: footprint ultim8x8_libs:APA102_U05 -> ultim8x64_libs:APA102
- U270, U278, U286, U302, U318: footprint ultim8x8_libs:APA102_U06 -> ultim8x64_libs:APA102
- U275: footprint ultim8x8_libs:APA102 -> ultim8x64_libs:APA102_U19
- U294: footprint ultim8x8_libs:APA102_U06 -> ultim8x64_libs:APA102_U38
- U299: footprint ultim8x8_libs:APA102 -> ultim8x64_libs:APA102_U43
- U309: footprint ultim8x8_libs:APA102_U05 -> ultim8x64_libs:APA102_U53
- U310: footprint ultim8x8_libs:APA102_U06 -> ultim8x64_libs:APA102_U54
- U315: footprint ultim8x8_libs:APA102 -> ultim8x64_libs:APA102_U59
- U316: footprint ultim8x8_libs:APA102 -> ultim8x64_libs:APA102_U60
Connections:
- net 5V: now also C17.1 (+), C18.1 (+), C19.1, C20.1, P9.1
- net GND: now also C17.2 (-), C18.2 (-), C19.2, C20.2, P10.1
Other:
- note added: "POWER INPUT POSTS"
