File: kicad/Row_F.sch (KiCad schematic (older format))
At the start: 68 parts, among them U321 APA102, U322 APA102, U323 APA102, U324 APA102, U325 APA102, U326 APA102, U327 APA102, U328 APA102, U329 APA102, U330 APA102, U331 APA102, U332 APA102, U333 APA102, U334 APA102, U335 APA102, U336 APA102, U337 APA102, U338 APA102, U339 APA102, U340 APA102, U341 APA102, U342 APA102, U343 APA102, U344 APA102, U345 APA102, U346 APA102, U347 APA102, U348 APA102, U349 APA102, U350 APA102, U351 APA102, U352 APA102, U353 APA102, U354 APA102, U355 APA102, U356 APA102, U357 APA102, U358 APA102, U359 APA102, U360 APA102, U361 APA102, U362 APA102, U363 APA102, U364 APA102, U365 APA102, U366 APA102, U367 APA102, U368 APA102, U369 APA102, U370 APA102, U371 APA102, U372 APA102, U373 APA102, U374 APA102, U375 APA102, U376 APA102, U377 APA102, U378 APA102, U379 APA102, U380 APA102, U381 APA102, U382 APA102, U383 APA102, U384 APA102

Commit message: WIP
Parts:
- C21, C22: footprint ultim8x8_libs:c_2917 -> ultim8x64_libs:c_2917
- C23, C24: footprint ultim8x8_libs:c_0805 -> ultim8x64_libs:c_0805
- U321, U322, U323, U324, U325, U326, U327, U328, U329, U330, U331, U332, U335, U336, U337, U338, U339, U340, U343, U344, U345, U346, U347, U348, U351, U352, U353, U354, U355, U356, U359, U360, U361, U362, U363, U364, U367, U368, U369, U370, U371, U372, U375, U376, U377, U378, U379, U380, U383, U384: footprint ultim8x8_libs:APA102 -> ultim8x64_libs:APA102
- U333, U341, U349, U357, U365, U373, U381: footprint ultim8x8_libs:APA102_U05 -> ultim8x64_libs:APA102
- U334, U342, U350, U358, U366, U374, U382: footprint ultim8x8_libs:APA102_U06 -> ultim8x64_libs:APA102
