File: kicad/Row_G.sch (KiCad schematic (older format))
At the start: 68 parts, among them U385 APA102, U386 APA102, U387 APA102, U388 APA102, U389 APA102, U390 APA102, U391 APA102, U392 APA102, U393 APA102, U394 APA102, U395 APA102, U396 APA102, U397 APA102, U398 APA102, U399 APA102, U400 APA102, U401 APA102, U402 APA102, U403 APA102, U404 APA102, U405 APA102, U406 APA102, U407 APA102, U408 APA102, U409 APA102, U410 APA102, U411 APA102, U412 APA102, U413 APA102, U414 APA102, U415 APA102, U416 APA102, U417 APA102, U418 APA102, U419 APA102, U420 APA102, U421 APA102, U422 APA102, U423 APA102, U424 APA102, U425 APA102, U426 APA102, U427 APA102, U428 APA102, U429 APA102, U430 APA102, U431 APA102, U432 APA102, U433 APA102, U434 APA102, U435 APA102, U436 APA102, U437 APA102, U438 APA102, U439 APA102, U440 APA102, U441 APA102, U442 APA102, U443 APA102, U444 APA102, U445 APA102, U446 APA102, U447 APA102, U448 APA102

Commit message: WIP
Parts:
- added P11: GND, ultim8x64_libs:PowerIn_stud, symbol CONN_1
- added P12: 5V, ultim8x64_libs:PowerIn_stud, symbol CONN_1
- C25, C26: footprint ultim8x8_libs:c_2917 -> ultim8x64_libs:c_2917
- C27, C28: footprint ultim8x8_libs:c_0805 -> ultim8x64_libs:c_0805
- U385, U386, U387, U388, U391, U392, U393, U394, U399, U400, U401, U402, U404, U407, U408, U409, U410, U411, U412, U415, U416, U417, U418, U419, U420, U423, U424, U425, U426, U428, U431, U432, U433, U434, U435, U436, U439, U440, U441, U442, U447, U448: footprint ultim8x8_libs:APA102 -> ultim8x64_libs:APA102
- U389: footprint ultim8x8_libs:APA102 -> ultim8x64_libs:APA102_U05
- U390: footprint ultim8x8_libs:APA102 -> ultim8x64_libs:APA102_U06
- U395: footprint ultim8x8_libs:APA102 -> ultim8x64_libs:APA102_U11
- U396: footprint ultim8x8_libs:APA102 -> ultim8x64_libs:APA102_U12
- U397, U405, U413, U421, U429, U445: footprint ultim8x8_libs:APA102_U05 -> ultim8x64_libs:APA102
- U398, U406, U414, U430, U446: footprint ultim8x8_libs:APA102_U06 -> ultim8x64_libs:APA102
- U403: footprint ultim8x8_libs:APA102 -> ultim8x64_libs:APA102_U19
- U422: footprint ultim8x8_libs:APA102_U06 -> ultim8x64_libs:APA102_U38
- U427: footprint ultim8x8_libs:APA102 -> ultim8x64_libs:APA102_U43
- U437: footprint ultim8x8_libs:APA102_U05 -> ultim8x64_libs:APA102_U53
- U438: footprint ultim8x8_libs:APA102_U06 -> ultim8x64_libs:APA102_U54
- U443: footprint ultim8x8_libs:APA102 -> ultim8x64_libs:APA102_U59
- U444: footprint ultim8x8_libs:APA102 -> ultim8x64_libs:APA102_U60
Connections:
- net 5V: now also C25.1 (+), C26.1 (+), C27.1, C28.1, P11.1
- net GND: now also C25.2 (-), C26.2 (-), C27.2, C28.2, P12.1
Other:
- note added: "POWER INPUT POSTS"
