File: kicad/Row_H.sch (KiCad schematic (older format))
At the start: 68 parts, among them U449 APA102, U450 APA102, U451 APA102, U452 APA102, U453 APA102, U454 APA102, U455 APA102, U456 APA102, U457 APA102, U458 APA102, U459 APA102, U460 APA102, U461 APA102, U462 APA102, U463 APA102, U464 APA102, U465 APA102, U466 APA102, U467 APA102, U468 APA102, U469 APA102, U470 APA102, U471 APA102, U472 APA102, U473 APA102, U474 APA102, U475 APA102, U476 APA102, U477 APA102, U478 APA102, U479 APA102, U480 APA102, U481 APA102, U482 APA102, U483 APA102, U484 APA102, U485 APA102, U486 APA102, U487 APA102, U488 APA102, U489 APA102, U490 APA102, U491 APA102, U492 APA102, U493 APA102, U494 APA102, U495 APA102, U496 APA102, U497 APA102, U498 APA102, U499 APA102, U500 APA102, U501 APA102, U502 APA102, U503 APA102, U504 APA102, U505 APA102, U506 APA102, U507 APA102, U508 APA102, U509 APA102, U510 APA102, U511 APA102, U512 APA102

Commit message: WIP
Parts:
- C29, C30: footprint ultim8x8_libs:c_2917 -> ultim8x64_libs:c_2917
- C31, C32: footprint ultim8x8_libs:c_0805 -> ultim8x64_libs:c_0805
- U449, U450, U451, U452, U453, U454, U455, U456, U457, U458, U459, U460, U463, U464, U465, U466, U467, U468, U471, U472, U473, U474, U475, U476, U479, U480, U481, U482, U483, U484, U487, U488, U489, U490, U491, U492, U495, U496, U497, U498, U499, U500, U503, U504, U505, U506, U507, U508, U511, U512: footprint ultim8x8_libs:APA102 -> ultim8x64_libs:APA102
- U461, U469, U477, U485, U493, U501, U509: footprint ultim8x8_libs:APA102_U05 -> ultim8x64_libs:APA102
- U462, U470, U478, U486, U494, U502, U510: footprint ultim8x8_libs:APA102_U06 -> ultim8x64_libs:APA102
