File: kicad/ultim8x64.sch (KiCad schematic (older format))
At the start: 10 parts, among them P1 Input1, P2 Output1, P3 Input2, P4 Output2, P5 5V, P6 GND

Commit message: WIP
Parts:
- removed P5: 5V, ultim8x8_libs:PowerIn_stud, symbol CONN_1
- removed P6: GND, ultim8x8_libs:PowerIn_stud, symbol CONN_1
- L2: footprint ultim8x8_libs:OSHW_6mm -> ultim8x64_libs:OSHW_6mm
- L3: footprint ultim8x8_libs:logo_wyo_butterfly -> ultim8x64_libs:logo_wyo_butterfly
- L4: footprint ultim8x8_libs:logo_MLlabs -> ultim8x64_libs:logo_MLlabs
- P1, P2, P3, P4: footprint ultim8x8_libs:header_3pos_smd_male -> ultim8x64_libs:header_3pos_smd_male
Other:
- note added: "POWER"
- note removed: "POWER INPUT POSTS"
Changed lines of the file:
@@
 F 0 "L2" V 1425 6600 40  0000 C CNN
 F 1 "OSHW" V 1225 6600 30  0000 C CNN
-F 2 "ultim8x8_libs:OSHW_6mm" H 1325 6755 30  0001 C CNN
+F 2 "ultim8x64_libs:OSHW_6mm" H 1325 6755 30  0001 C CNN
 F 3 "" H 1325 6600 60  0001 C CNN
 	1    1325 6600
@@
 F 0 "L3" V 1775 6600 40  0000 C CNN
 F 1 "Wyolum" V 1575 6600 30  0000 C CNN
-F 2 "ultim8x8_libs:logo_wyo_butterfly" H 1600 6675 30  0001 C CNN
+F 2 "ultim8x64_libs:logo_wyo_butterfly" H 1600 6675 30  0001 C CNN
 F 3 "" H 1675 6600 60  0001 C CNN
 	1    1675 6600
@@
 $EndSheet
 $Comp
-L PWR_FLAG #FLG1
+L PWR_FLAG #FLG01
 U 1 1 50E7FAAF
 P 1375 4150
-F 0 "#FLG1" H 1375 4245 30  0001 C CNN
+F 0 "#FLG01" H 1375 4245 30  0001 C CNN
 F 1 "PWR_FLAG" H 1375 4330 30  0000 C CNN
 F 2 "" H 1375 4150 60  0001 C CNN
@@
 	1    0    0    -1
 $EndComp
-Text Label 1875 4300 0    60   ~ 0
+Text Label 1875 4150 0    60   ~ 12
 5V
 Text Label 1550 2100 2    40   ~ 0
@@
 CI_A
 $Comp
-L GND #PWR1
+L GND #PWR02
 U 1 1 56C3FF09
 P 1375 4900
-F 0 "#PWR1" H 1375 4650 50  0001 C CNN
+F 0 "#PWR02" H 1375 4650 50  0001 C CNN
 F 1 "GND" H 1375 4750 50  0000 C CNN
 F 2 "" H 1375 4900 50  0000 C CNN
@@
 	1    0    0    -1
 $EndComp
-Text Label 1875 4800 0    60   ~ 0
+Text Label 1875 4650 0    60   ~ 12
 GND
 $Comp
-L PWR_FLAG #FLG2
+L PWR_FLAG #FLG03
 U 1 1 56C40925
 P 1375 4650
-F 0 "#FLG2" H 1375 4745 30  0001 C CNN
+F 0 "#FLG03" H 1375 4745 30  0001 C CNN
 F 1 "PWR_FLAG" H 1375 4830 30  0000 C CNN
 F 2 "" H 1375 4650 60  0001 C CNN
@@
 F 0 "P1" H 1025 1325 40  0000 C CNB
 F 1 "Input1" H 1000 1725 40  0000 C CNN
-F 2 "ultim8x8_libs:header_3pos_smd_male" H 1000 1475 60  0001 C CNN
+F 2 "ultim8x64_libs:header_3pos_smd_male" H 1000 1475 60  0001 C CNN
 F 3 "" H 1000 1475 60  0000 C CNN
 F 4 "CONN HEADER 50POS .100\" SGL GOLD" H 1000 1575 60  0001 L CNN "Field4"
@@
 F 0 "P2" H 2350 1725 40  0000 C CNB
 F 1 "Output1" H 2350 1325 40  0000 C CNN
-F 2 "ultim8x8_libs:header_3pos_smd_male" H 2350 1475 60  0001 C CNN
+F 2 "ultim8x64_libs:header_3pos_smd_male" H 2350 1475 60  0001 C CNN
 F 3 "" H 2350 1475 60  0000 C CNN
 F 4 "CONN HEADER 50POS .100\" SGL GOLD" H 2350 1575 60  0001 L CNN "Field4"
@@
 F 0 "P3" H 1000 2000 40  0000 C CNB
 F 1 "Input2" H 1000 2400 40  0000 C CNN
-F 2 "ultim8x8_libs:header_3pos_smd_male" H 1000 2150 60  0001 C CNN
+F 2 "ultim8x64_libs:header_3pos_smd_male" H 1000 2150 60  0001 C CNN
 F 3 "" H 1000 2150 60  0000 C CNN
 F 4 "CONN HEADER 50POS .100\" SGL GOLD" H 1000 2250 60  0001 L CNN "Field4"
@@
 F 0 "P4" H 2350 2400 40  0000 C CNB
 F 1 "Output2" H 2350 2000 40  0000 C CNN
-F 2 "ultim8x8_libs:header_3pos_smd_male" H 2350 2150 60  0001 C CNN
+F 2 "ultim8x64_libs:header_3pos_smd_male" H 2350 2150 60  0001 C CNN
 F 3 "" H 2350 2150 60  0000 C CNN
 F 4 "CONN HEADER 50POS .100\" SGL GOLD" H 2350 2250 60  0001 L CNN "Field4"
@@
 Text Label 6475 5900 2    60   ~ 0
 CI_H
-$Comp
-L CONN_1 P5
-U 1 1 56C23A5D
-P 1700 4025
-F 0 "P5" V 1775 3950 40  0000 L CNB
-F 1 "5V" H 1700 4080 30  0001 C CNN
-F 2 "ultim8x8_libs:PowerIn_stud" H 1700 4025 60  0001 C CNN
-F 3 "" H 1700 4025 60  0000 C CNN
-F 4 "mfr_pn" H 1700 4025 60  0001 C CNN "manf#"
-	1    1700 4025
-	0    -1   -1   0
-$EndComp
-$Comp
-L CONN_1 P6
-U 1 1 56C2406F
-P 1700 4525
-F 0 "P6" V 1775 4450 40  0000 L CNB
-F 1 "GND" H 1700 4580 30  0001 C CNN
-F 2 "ultim8x8_libs:PowerIn_stud" H 1700 4525 60  0001 C CNN
-F 3 "" H 1700 4525 60  0000 C CNN
-F 4 "mfr_pn" H 1700 4525 60  0001 C CNN "manf#"
-	1    1700 4525
-	0    -1   -1   0
-$EndComp
 Text Notes 700  6100 0    60   ~ 12
 LOGOS
 Text Notes 700  3500 0    60   ~ 12
-POWER INPUT POSTS
+POWER
 Text Notes 2000 2700 0    60   ~ 12
 DATA/CLK\nOUTPUTS
@@
 F 0 "L4" V 2125 6600 40  0000 C CNN
 F 1 "Maniacal Labs" V 1925 6600 30  0000 C CNN
-F 2 "ultim8x8_libs:logo_MLlabs" H 1950 6675 30  0001 C CNN
+F 2 "ultim8x64_libs:logo_MLlabs" H 1950 6675 30  0001 C CNN
 F 3 "" H 2025 6600 60  0001 C CNN
 	1    2025 6600
@@
 60 BD D6 69 7C FA 84 4E 00 1C F3 6D BF C6 02 A0 13 00 C7 7C AB 8B FD F9 43 66 C3 B0 78 D8 F1 6E
 2F 80 9D 81 10 24 E6 C1 CF 81 0B 01 EC D4 00 18 4E AC 7F 37 5C 08 FB CB C7 8F 46 91 1C 94 52 FC
-EC F0 FD 0F 88 A0 E4 D1 04 AE BA DB 00 00 00 00 49 45 4E 44 AE 42 60 82 A1
+EC F0 FD 0F 88 A0 E4 D1 04 AE BA DB 00 00 00 00 49 45 4E 44 AE 42 60 82 01
 EndData
 $EndBitmap
@@
 	5925 6500 6475 6500
 Wire Wire Line
-	1375 4300 1700 4300
-Wire Wire Line
-	1700 4300 1875 4300
+	1375 4300 1875 4300
 Wire Wire Line
 	1375 4150 1375 4300
@@
 	1550 2200 1350 2200
 Wire Wire Line
-	1875 4800 1700 4800
-Wire Wire Line
-	1700 4800 1375 4800
-Wire Wire Line
-	1375 4650 1375 4800
-Wire Wire Line
-	1375 4800 1375 4900
+	1375 4800 1875 4800
+Wire Wire Line
+	1375 4650 1375 4900
 Connection ~ 1375 4800
-Wire Wire Line
-	1700 4175 1700 4300
-Connection ~ 1700 4300
-Wire Wire Line
-	1700 4675 1700 4800
-Connection ~ 1700 4800
 Wire Notes Line
 	700  900  2700 900
@@
 F7 "5V" I R 5925 6800 50
 $EndSheet
+Wire Wire Line
+	1875 4300 1875 4150
+Wire Wire Line
+	1875 4800 1875 4650
 $EndSCHEMATC
